Commit message: Created max_dev branch

File: ros2_ws/src/modproft_camera_description/urdf/_camera.urdf.xacro (robot description, xacro)
@@ -2,5 +2,5 @@
 <robot xmlns:xacro="http://wiki.ros.org/xacro" name="camera_test">
    <!-- import macro-->
-   <xacro:include filename="$(find modproft_camera_description)/urdf/camera_macro_depreached.xacro"/>
+   <xacro:include filename="$(find modproft_camera_description)/urdf/camera_macro.xacro"/>
    <!-- create link fixed to the "world" -->
    <link name="world" />

File: ros2_ws/src/modproft_camera_description/urdf/camera_macro.xacro (robot description, xacro)
@@ -1,52 +1,50 @@
 <?xml version="1.0"?>
 <robot xmlns:xacro="http://wiki.ros.org/xacro">
-  <xacro:arg name="package_name" default="modproft_camera_description" />
-  <xacro:property name="package_name" value="$(arg package_name)" />
-  <xacro:property name="camera_type" value="canon_powershot_g7_mk3" />
-  <xacro:include filename="$(find ${package_name})/urdf/inc/camera_common.xacro" />
-  <xacro:read_camera_data model_parameter_file="$(find ${package_name})/config/${camera_type}.yaml"/>
-  <xacro:macro name="generate_camera" params="prefix attachment_link">
+   <xacro:macro name="generate_camera" params="prefix attachment_link package_name:=modproft_camera_description camera_type:=canon_powershot_g7_mk3">
+    <xacro:include filename="$(find ${package_name})/urdf/inc/camera_common.xacro"/>
+    <xacro:include filename="$(find ${package_name})/urdf/inc/materials.xacro"/>
+    <xacro:read_camera_data model_parameter_file="$(find ${package_name})/config/${camera_type}.yaml"/>
     <!-- Define gazebo sensor -->
-      <gazebo reference="${prefix}camera_link">
-        <sensor type="${sensor_type}" name="${prefix}camera">
-          <always_on>${sensor_always_on}</always_on>
-          <update_rate>${sensor_update_rate}</update_rate>
-          <camera name="${sensor_name}">
-            <horizontal_fov>${sensor_horizontal_fov}</horizontal_fov>
-            <image>
-              <width>${sensor_image_width}</width>
-              <height>${sensor_image_height}</height>
-              <format>${sensor_image_format}</format>
-            </image>
-            <clip>
-              <near>${sensor_image_clip_near}</near>
-              <far>${sensor_image_clip_far}</far>
-            </clip>
-            <distortion>
-              <k1>${sensor_image_distortion_k1}</k1>
-              <k2>${sensor_image_distortion_k2}</k2>
-              <k3>${sensor_image_distortion_k3}</k3>
-              <p1>${sensor_image_distortion_p1}</p1>
-              <p2>${sensor_image_distortion_p2}</p2>
-              <center>${sensor_image_distortion_center}</center>
-            </distortion>
-          </camera>
-          <plugin name="${prefix}_${sensor_name}_camera_controller" filename="libgazebo_ros_camera.so">
-            <ros>
-              <imageTopicName>${prefix}/${sensor_name}/color/image_raw</imageTopicName>
-              <cameraInfoTopicName>${prefix}/${sensor_name}/color/camera_info</cameraInfoTopicName>
-              <depthImageTopicName>${prefix}/${sensor_name}/depth/image_raw</depthImageTopicName>
-              <depthImageCameraInfoTopicName>${prefix}/${sensor_name}/depth/camera_info</depthImageCameraInfoTopicName>
-              <pointCloudTopicName>${prefix}/${sensor_name}/depth/points</pointCloudTopicName>
-            </ros>
-            <camera_name>${prefix}_${sensor_name}_camera</camera_name>
-            <frame_name>${prefix}camera_link</frame_name>
-            <hack_baseline>${sensor_hack_baseline}</hack_baseline>
-            <min_depth>${sensor_min_depth}</min_depth>
-          </plugin>
-        </sensor>
-      </gazebo>
+    <gazebo reference="${prefix}${sensor_name}_link">
+      <sensor name="${prefix}${sensor_name}" type="${sensor_type}" >
+        <always_on>${sensor_always_on}</always_on>
+        <update_rate>${sensor_update_rate}</update_rate>
+        <camera name="${prefix}${sensor_name}">
+          <horizontal_fov>${sensor_horizontal_fov}</horizontal_fov>
+          <image>
+            <width>${sensor_image_width}</width>
+            <height>${sensor_image_height}</height>
+            <format>${sensor_image_format}</format>
+          </image>
+          <clip>
+            <near>${sensor_image_clip_near}</near>
+            <far>${sensor_image_clip_far}</far>
+          </clip>
+          <distortion>
+            <k1>${sensor_image_distortion_k1}</k1>
+            <k2>${sensor_image_distortion_k2}</k2>
+            <k3>${sensor_image_distortion_k3}</k3>
+            <p1>${sensor_image_distortion_p1}</p1>
+            <p2>${sensor_image_distortion_p2}</p2>
+            <center>${sensor_image_distortion_center}</center>
+          </distortion>
+        </camera>
+        <plugin filename="libgazebo_ros_camera.so" name="${prefix}${sensor_name}_controller">
+          <ros>
+            <imageTopicName>/${prefix}${sensor_name}/color/image_raw</imageTopicName>
+            <cameraInfoTopicName>/${prefix}${sensor_name}/color/camera_info</cameraInfoTopicName>
+            <depthImageTopicName>/${prefix}${sensor_name}/depth/image_raw</depthImageTopicName>
+            <depthImageCameraInfoTopicName>/${prefix}${sensor_name}/depth/camera_info</depthImageCameraInfoTopicName>
+            <pointCloudTopicName>/${prefix}${sensor_name}/depth/points</pointCloudTopicName>
+          </ros>
+          <camera_name>${prefix}${sensor_name}</camera_name>
+          <frame_name>${prefix}${sensor_name}_link</frame_name>
+          <hack_baseline>${sensor_hack_baseline}</hack_baseline>
+          <min_depth>${sensor_min_depth}</min_depth>
+        </plugin>
+      </sensor>
+    </gazebo>
     <!-- Links -->
-    <link name="${prefix}camera_link">
+    <link name="${prefix}${sensor_name}_link">
       <visual>
         <origin rpy="${camera_visual_origin_rpy}" xyz="${camera_visual_origin_xyz}"/>
@@ -69,9 +67,9 @@
     </link>
     <!-- Joints -->
-    <joint type="fixed" name="${prefix}${attachment_link}_camera_joint">
-      <origin rpy="-1.57 0.0 0.0" xyz="${cameraattachment_joint_origin_xyz}"/>
-      <child link="${prefix}camera_link"/>
+    <joint type="fixed" name="${prefix}${attachment_link}_${sensor_name}_joint">
+      <origin rpy="${cameraattachment_joint_origin_rpy}" xyz="${cameraattachment_joint_origin_xyz}"/>
+      <child link="${prefix}${sensor_name}_link"/>
       <parent link="${prefix}${attachment_link}"/>
     </joint>
- </xacro:macro>
+  </xacro:macro>
 </robot>

File: ros2_ws/src/modproft_camera_description/urdf/camera_macro_depreached.xacro (robot description, xacro)
@@ -32,5 +32,5 @@
               <cameraInfoTopicName>${prefix}/camera/color/camera_info</cameraInfoTopicName>
               <depthImageTopicName>${prefix}/camera/depth/image_raw</depthImageTopicName>
-              <depthImageCameraInfoTopicName>${prefix}/camera/depth/camera_info</depthImageCameraInfoTopicName>
+              <depthImageCameraInfoTopicName>/${prefix}/camera/depth/camera_info</depthImageCameraInfoTopicName>
               <pointCloudTopicName>${prefix}/camera/depth/points</pointCloudTopicName>
             </ros>
@@ -68,4 +68,5 @@
       <parent link="${prefix}${attachment_link}"/>
     </joint>
- </xacro:macro>
+  </xacro:macro>
+  <xacro:generate_camera prefix="" attachment_link="tool0"/>
 </robot>

File: ros2_ws/src/modproft_ur_description/urdf/ur.urdf.xacro (robot description, xacro)
@@ -4,5 +4,5 @@
    <xacro:include filename="$(find ur_description)/urdf/ur_macro.xacro"/>
    <!-- <xacro:include filename="$(find modproft_camera_description)/urdf/camera_macro.xacro"/> -->
-   <xacro:include filename="$(find modproft_camera_description)/urdf/camera_macro_depreached.xacro"/>
+   <xacro:include filename="$(find modproft_camera_description)/urdf/camera_macro.xacro"/>
    <!-- robot definition -->
    <!-- possible 'ur_type' values: ur3, ur3e, ur5, ur5e, ur10, ur10e, ur16e -->
