Commit message: Camera direction fixed; Octomap fixed; Context added to ur_movit.launch; User permission problems fixed;

File: ros2_ws/src/modproft_camera_description/urdf/camera_macro.xacro (robot description, xacro)
@@ -1,14 +1,23 @@
 <?xml version="1.0"?>
 <robot xmlns:xacro="http://wiki.ros.org/xacro">
-   <xacro:macro name="generate_camera" params="prefix attachment_link package_name:=modproft_camera_description camera_type:=canon_powershot_g7_mk3">
+   <xacro:macro name="generate_camera" params="prefix attachment_link package_name:=modproft_camera_description camera_type:=canon_powershot_g7_mk3 debug:=False">
     <xacro:include filename="$(find ${package_name})/urdf/inc/camera_common.xacro"/>
     <xacro:include filename="$(find ${package_name})/urdf/inc/materials.xacro"/>
     <xacro:read_camera_data model_parameter_file="$(find ${package_name})/config/${camera_type}.yaml"/>
+    <xacro:property name="prefix_default" value=""/>
+    <xacro:property name="debug_enabled" value="False"/>
+    <!-- Todo: Fix Prefix ${prefix} != &quot; &quot;-->
+    <xacro:if value="${prefix != prefix_default}">
+      <xacro:property name="sensor_reference" value="${prefix}${sensor_name}"/>
+    </xacro:if>
+    <xacro:if value="${prefix == prefix_default}">
+      <xacro:property name="sensor_reference" value="${sensor_name}"/>
+    </xacro:if>
     <!-- Define gazebo sensor -->
-    <gazebo reference="${prefix}${sensor_name}_link">
-      <sensor name="${prefix}${sensor_name}" type="${sensor_type}" >
+    <gazebo reference="${sensor_reference}_link">
+      <sensor name="${sensor_reference}" type="${sensor_type}" >
         <always_on>${sensor_always_on}</always_on>
         <update_rate>${sensor_update_rate}</update_rate>
-        <camera name="${prefix}${sensor_name}">
+        <camera name="${sensor_reference}">
           <horizontal_fov>${sensor_horizontal_fov}</horizontal_fov>
           <image>
@@ -30,14 +39,14 @@
           </distortion>
         </camera>
-        <plugin filename="libgazebo_ros_camera.so" name="${prefix}${sensor_name}_controller">
+        <plugin filename="libgazebo_ros_camera.so" name="${sensor_reference}_controller">
           <ros>
-            <imageTopicName>/${prefix}${sensor_name}/color/image_raw</imageTopicName>
-            <cameraInfoTopicName>/${prefix}${sensor_name}/color/camera_info</cameraInfoTopicName>
-            <depthImageTopicName>/${prefix}${sensor_name}/depth/image_raw</depthImageTopicName>
-            <depthImageCameraInfoTopicName>/${prefix}${sensor_name}/depth/camera_info</depthImageCameraInfoTopicName>
-            <pointCloudTopicName>/${prefix}${sensor_name}/depth/points</pointCloudTopicName>
+              <imageTopicName>/${sensor_reference}/color/image_raw</imageTopicName>
+              <cameraInfoTopicName>/${sensor_reference}/color/camera_info</cameraInfoTopicName>
+              <depthImageTopicName>/${sensor_reference}/depth/image_raw</depthImageTopicName>
+              <depthImageCameraInfoTopicName>/${sensor_reference}/depth/camera_info</depthImageCameraInfoTopicName>
+              <pointCloudTopicName>/${sensor_reference}/points</pointCloudTopicName>
           </ros>
-          <camera_name>${prefix}${sensor_name}</camera_name>
-          <frame_name>${prefix}${sensor_name}_link</frame_name>
+          <camera_name>${sensor_reference}</camera_name>
+          <frame_name>${sensor_reference}_virtual_frame_link</frame_name>
           <hack_baseline>${sensor_hack_baseline}</hack_baseline>
           <min_depth>${sensor_min_depth}</min_depth>
@@ -46,5 +55,5 @@
     </gazebo>
     <!-- Links -->
-    <link name="${prefix}${sensor_name}_link">
+    <link name="${sensor_reference}_link">
       <visual>
         <origin rpy="${camera_visual_origin_rpy}" xyz="${camera_visual_origin_xyz}"/>
@@ -66,9 +75,24 @@
       </inertial>
     </link>
+    <link name="${sensor_reference}_virtual_frame_link">
+      <!-- Todo Fix debug condition block-->
+      <xacro:if value="${debug != debug_enabled}">
+        <visual>
+          <geometry>
+            <mesh filename="package://${package_name}/meshes/${virtual_visual_geometry_mesh}" scale="${virtual_visual_geometry_scale}"/>
+          </geometry>
+        </visual>
+      </xacro:if>
+    </link>
     <!-- Joints -->
     <joint type="fixed" name="${prefix}${attachment_link}_${sensor_name}_joint">
       <origin rpy="${cameraattachment_joint_origin_rpy}" xyz="${cameraattachment_joint_origin_xyz}"/>
-      <child link="${prefix}${sensor_name}_link"/>
+      <child link="${sensor_reference}_link"/>
       <parent link="${prefix}${attachment_link}"/>
+    </joint>
+    <joint type="fixed" name="${prefix}${attachment_link}_${sensor_name}_virtual_frame_joint">
+      <origin rpy="${cameravirtual_joint_origin_rpy}" xyz="${cameravirtual_joint_origin_xyz}"/>
+      <child link="${sensor_reference}_virtual_frame_link"/>
+      <parent link="${sensor_reference}_link"/>
     </joint>
   </xacro:macro>

File: ros2_ws/src/modproft_camera_description/urdf/inc/camera_common.xacro (robot description, xacro)
@@ -24,4 +24,6 @@
         <xacro:property name="camera_visual_geometry_scale" value="${camera['visual']['geometry']['scale']}" scope="parent"/>
         <xacro:property name="camera_visual_material" value="${camera['visual']['material']}" scope="parent"/>
+        <xacro:property name="virtual_visual_geometry_mesh" value="${camera['virtual']['visual']['geometry']['mesh']}" scope="parent"/>
+        <xacro:property name="virtual_visual_geometry_scale" value="${camera['virtual']['visual']['geometry']['scale']}" scope="parent"/>
         <!-- Collision parameters -->
         <xacro:property name="camera_collision_origin_rpy" value="${camera['collision']['origin']['rpy']}" scope="parent"/>
@@ -48,7 +50,9 @@
         <xacro:property name="sensor_hack_baseline" value="${camera['sensor']['hack_baseline']}" scope="parent"/>
         <xacro:property name="sensor_min_depth" value="${camera['sensor']['min_depth']}" scope="parent"/>
-        <!-- Joint -->
+        <!-- Joints -->
         <xacro:property name="cameraattachment_joint_origin_rpy" value="${camera['joints']['attachment_joint']['origin']['rpy']}" scope="parent"/>
         <xacro:property name="cameraattachment_joint_origin_xyz" value="${camera['joints']['attachment_joint']['origin']['xyz']}" scope="parent"/>
+        <xacro:property name="cameravirtual_joint_origin_rpy" value="${camera['joints']['virtual_joint']['origin']['rpy']}" scope="parent"/>
+        <xacro:property name="cameravirtual_joint_origin_xyz" value="${camera['joints']['virtual_joint']['origin']['xyz']}" scope="parent"/>
     </xacro:macro>
 </robot>

Commit message: Adding manipulator, tables; adapting collisons

File: ros2_ws/src/modproft_camera_description/urdf/camera_macro.xacro (robot description, xacro)
@@ -3,5 +3,6 @@
    <xacro:macro name="generate_camera" params="prefix attachment_link package_name:=modproft_camera_description camera_type:=canon_powershot_g7_mk3 debug:=False">
     <xacro:include filename="$(find ${package_name})/urdf/inc/camera_common.xacro"/>
-    <xacro:include filename="$(find ${package_name})/urdf/inc/materials.xacro"/>
+    <!-- Uncomment for in-package colors -->
+    <!--<xacro:include filename="$(find ${package_name})/urdf/inc/materials.xacro"/>-->
     <xacro:read_camera_data model_parameter_file="$(find ${package_name})/config/${camera_type}.yaml"/>
     <xacro:property name="prefix_default" value=""/>
@@ -66,5 +67,7 @@
           <mesh filename="package://${package_name}/meshes/${camera_visual_geometry_mesh}" scale="${camera_visual_geometry_scale}"/>
         </geometry>
-        <material name="${camera_visual_material}"/>
+        <!-- Uncomment for in-package colors -->
+        <!--<material name="${camera_visual_material}"/>-->
+        <xacro:material_silver/>
       </collision>
       <inertial>

File: ros2_ws/src/modproft_manipulator_description/urdf/manipulator_macro.xacro (robot description, xacro)
@@ -3,5 +3,6 @@
    <xacro:macro name="generate_manipulator" params="prefix attachment_link manipulator_name package_name:=modproft_manipulator_description manipulator_type:=manipulator_klinke_v2">
     <xacro:include filename="$(find ${package_name})/urdf/inc/manipulator_common.xacro"/>
-    <xacro:include filename="$(find ${package_name})/urdf/inc/materials.xacro"/>
+    <!-- Uncomment for in-package colors -->
+    <!--<xacro:include filename="$(find ${package_name})/urdf/inc/materials.xacro"/>-->
     <xacro:read_manipulator_data model_parameter_file="$(find ${package_name})/config/${manipulator_type}.yaml"/>
     <xacro:property name="prefix_default" value=""/>
@@ -26,5 +27,7 @@
           <mesh filename="package://${package_name}/meshes/${manipulator_visual_geometry_mesh}" scale="${manipulator_visual_geometry_scale}"/>
         </geometry>
-        <material name="${manipulator_visual_material}"/>
+        <!-- Uncomment for in-package colors -->
+        <!--<material name="${manipulator_visual_material}"/>-->
+        <xacro:material_silver/>
       </collision>
       <inertial>

File: ros2_ws/src/modproft_table_description/urdf/inc/materials.xacro (robot description, xacro)
@@ -1,4 +1,4 @@
 <?xml version="1.0" ?>
-<robot name="manipulator" xmlns:xacro="http://www.ros.org/wiki/xacro" >
+<robot name="table" xmlns:xacro="http://www.ros.org/wiki/xacro" >
 <material name="silver">
   <color rgba="0.700 0.700 0.700 1.000"/>

File: ros2_ws/src/modproft_ur_description/urdf/ur.urdf.xacro (robot description, xacro)
@@ -1,90 +1,91 @@
 <?xml version="1.0"?>
 <robot xmlns:xacro="http://wiki.ros.org/xacro" name="$(arg name)">
-   <!-- import macros-->
-   <xacro:include filename="$(find ur_description)/urdf/ur_macro.xacro"/>
-   <!-- <xacro:include filename="$(find modproft_camera_description)/urdf/camera_macro.xacro"/> -->
-   <xacro:include filename="$(find modproft_camera_description)/urdf/camera_macro.xacro"/>
-   <!-- robot definition -->
-   <!-- possible 'ur_type' values: ur3, ur3e, ur5, ur5e, ur10, ur10e, ur16e -->
-   <!-- the default value should raise an error in case this was called without defining the type -->
-   <xacro:arg name="ur_type" default="ur5x"/>
-   <!-- robot parameters -->
-   <xacro:arg name="name" default="ur"/>
-   <xacro:arg name="prefix" default="" />
-   <xacro:arg name="joint_limit_params" default="$(find ur_description)/config/$(arg ur_type)/joint_limits.yaml"/>
-   <xacro:arg name="kinematics_params" default="$(find ur_description)/config/$(arg ur_type)/default_kinematics.yaml"/>
-   <xacro:arg name="physical_params" default="$(find ur_description)/config/$(arg ur_type)/physical_parameters.yaml"/>
-   <xacro:arg name="visual_params" default="$(find ur_description)/config/$(arg ur_type)/visual_parameters.yaml"/>
-   <xacro:arg name="transmission_hw_interface" default=""/>
-   <xacro:arg name="safety_limits" default="false"/>
-   <xacro:arg name="safety_pos_margin" default="0.15"/>
-   <xacro:arg name="safety_k_position" default="20"/>
-   <!-- ros2_control related parameters -->
-   <xacro:arg name="headless_mode" default="false" />
-   <xacro:arg name="robot_ip" default="0.0.0.0" />
-   <xacro:arg name="script_filename" default=""/>
-   <xacro:arg name="output_recipe_filename" default=""/>
-   <xacro:arg name="input_recipe_filename" default=""/>
-   <!--   tool communication related parameters-->
-   <xacro:arg name="use_tool_communication" default="false" />
-   <xacro:arg name="tool_voltage" default="24" />
-   <xacro:arg name="tool_parity" default="0" />
-   <xacro:arg name="tool_baud_rate" default="115200" />
-   <xacro:arg name="tool_stop_bits" default="1" />
-   <xacro:arg name="tool_rx_idle_chars" default="1.5" />
-   <xacro:arg name="tool_tx_idle_chars" default="3.5" />
-   <xacro:arg name="tool_device_name" default="/tmp/ttyUR" />
-   <xacro:arg name="tool_tcp_port" default="54321" />
-     <!-- Simulation parameters -->
-   <xacro:arg name="use_fake_hardware" default="false" />
-   <xacro:arg name="fake_sensor_commands" default="false" />
-   <xacro:arg name="sim_gazebo" default="false" />
-   <xacro:arg name="sim_ignition" default="false" />
-   <xacro:arg name="simulation_controllers" default="" />
-   <!-- initial position for simulations (Fake Hardware, Gazebo, Ignition) -->
-   <xacro:arg name="initial_positions_file" default="$(find ur_description)/config/initial_positions.yaml"/>
-   <!-- convert to property to use substitution in function -->
-   <xacro:property name="initial_positions_file" default="$(arg initial_positions_file)"/>
-   <!-- create link fixed to the "world" -->
-   <link name="world" />
-   <!-- arm -->
-   <xacro:ur_robot
-     name="$(arg name)"
-     prefix="$(arg prefix)"
-     parent="world"
-     joint_limits_parameters_file="$(arg joint_limit_params)"
-     kinematics_parameters_file="$(arg kinematics_params)"
-     physical_parameters_file="$(arg physical_params)"
-     visual_parameters_file="$(arg visual_params)"
-     transmission_hw_interface="$(arg transmission_hw_interface)"
-     safety_limits="$(arg safety_limits)"
-     safety_pos_margin="$(arg safety_pos_margin)"
-     safety_k_position="$(arg safety_k_position)"
-     use_fake_hardware="$(arg use_fake_hardware)"
-     fake_sensor_commands="$(arg fake_sensor_commands)"
-     sim_gazebo="$(arg sim_gazebo)"
-     sim_ignition="$(arg sim_ignition)"
-     headless_mode="$(arg headless_mode)"
-     initial_positions="${load_yaml(initial_positions_file)}"
-     use_tool_communication="$(arg use_tool_communication)"
-     tool_voltage="$(arg tool_voltage)"
-     tool_parity="$(arg tool_parity)"
-     tool_baud_rate="$(arg tool_baud_rate)"
-     tool_stop_bits="$(arg tool_stop_bits)"
-     tool_rx_idle_chars="$(arg tool_rx_idle_chars)"
-     tool_tx_idle_chars="$(arg tool_tx_idle_chars)"
-     tool_device_name="$(arg tool_device_name)"
-     tool_tcp_port="$(arg tool_tcp_port)"
-     robot_ip="$(arg robot_ip)"
-     script_filename="$(arg script_filename)"
-     output_recipe_filename="$(arg output_recipe_filename)"
-     input_recipe_filename="$(arg input_recipe_filename)"
-     >
-     <origin xyz="0 0 0" rpy="0 0 0" />          <!-- position robot in the world -->
-   </xacro:ur_robot>
-   <xacro:if value="$(arg sim_gazebo)">
+  <!-- import macros-->
+  <xacro:include filename="$(find modproft_table_description)/urdf/table_macro.xacro" />
+  <xacro:include filename="$(find ur_description)/urdf/ur_macro.xacro" />
+  <xacro:include filename="$(find modproft_manipulator_description)/urdf/manipulator_macro.xacro" />
+  <xacro:include filename="$(find modproft_camera_description)/urdf/camera_macro.xacro" />
+  <xacro:include filename="$(find modproft_common)/urdf/common_material_macro.xacro"/>
+  <!-- robot definition -->
+  <!-- possible 'ur_type' values: ur3, ur3e, ur5, ur5e, ur10, ur10e, ur16e -->
+  <!-- the default value should raise an error in case this was called without defining the type -->
+  <xacro:arg name="ur_type" default="ur5x" />
+  <!-- robot parameters -->
+  <xacro:arg name="name" default="ur" />
+  <xacro:arg name="prefix" default="" />
+  <xacro:arg name="joint_limit_params" default="$(find ur_description)/config/$(arg ur_type)/joint_limits.yaml" />
+  <xacro:arg name="kinematics_params" default="$(find ur_description)/config/$(arg ur_type)/default_kinematics.yaml" />
+  <xacro:arg name="physical_params" default="$(find ur_description)/config/$(arg ur_type)/physical_parameters.yaml" />
+  <xacro:arg name="visual_params" default="$(find ur_description)/config/$(arg ur_type)/visual_parameters.yaml" />
+  <xacro:arg name="transmission_hw_interface" default="" />
+  <xacro:arg name="safety_limits" default="false" />
+  <xacro:arg name="safety_pos_margin" default="0.15" />
+  <xacro:arg name="safety_k_position" default="20" />
+  <!-- ros2_control related parameters -->
+  <xacro:arg name="headless_mode" default="false" />
+  <xacro:arg name="robot_ip" default="0.0.0.0" />
+  <xacro:arg name="script_filename" default="" />
+  <xacro:arg name="output_recipe_filename" default="" />
+  <xacro:arg name="input_recipe_filename" default="" />
+  <!--   tool communication related parameters-->
+  <xacro:arg name="use_tool_communication" default="false" />
+  <xacro:arg name="tool_voltage" default="24" />
+  <xacro:arg name="tool_parity" default="0" />
+  <xacro:arg name="tool_baud_rate" default="115200" />
+  <xacro:arg name="tool_stop_bits" default="1" />
+  <xacro:arg name="tool_rx_idle_chars" default="1.5" />
+  <xacro:arg name="tool_tx_idle_chars" default="3.5" />
+  <xacro:arg name="tool_device_name" default="/tmp/ttyUR" />
+  <xacro:arg name="tool_tcp_port" default="54321" />
+  <!-- Simulation parameters -->
+  <xacro:arg name="use_fake_hardware" default="false" />
+  <xacro:arg name="fake_sensor_commands" default="false" />
+  <xacro:arg name="sim_gazebo" default="false" />
+  <xacro:arg name="sim_ignition" default="false" />
+  <xacro:arg name="simulation_controllers" default="" />
+  <!-- initial position for simulations (Fake Hardware, Gazebo, Ignition) -->
+  <xacro:arg name="initial_positions_file" default="$(find modproft_ur_description)/config/initial_positions.yaml" />
+  <!-- convert to property to use substitution in function -->
+  <xacro:property name="initial_positions_file" default="$(arg initial_positions_file)" />
+  <!-- create link fixed to the "world" -->
+  <link name="world" />
+  <!-- arm -->
+  <xacro:ur_robot
+    name="$(arg name)"
+    prefix="$(arg prefix)"
+    parent="$(arg prefix)robot_table_tabletop_link"
+    joint_limits_parameters_file="$(arg joint_limit_params)"
+    kinematics_parameters_file="$(arg kinematics_params)"
+    physical_parameters_file="$(arg physical_params)"
+    visual_parameters_file="$(arg visual_params)"
+    transmission_hw_interface="$(arg transmission_hw_interface)"
+    safety_limits="$(arg safety_limits)"
+    safety_pos_margin="$(arg safety_pos_margin)"
+    safety_k_position="$(arg safety_k_position)"
+    use_fake_hardware="$(arg use_fake_hardware)"
+    fake_sensor_commands="$(arg fake_sensor_commands)"
+    sim_gazebo="$(arg sim_gazebo)"
+    sim_ignition="$(arg sim_ignition)"
+    headless_mode="$(arg headless_mode)"
+    initial_positions="${load_yaml(initial_positions_file)}"
+    use_tool_communication="$(arg use_tool_communication)"
+    tool_voltage="$(arg tool_voltage)"
+    tool_parity="$(arg tool_parity)"
+    tool_baud_rate="$(arg tool_baud_rate)"
+    tool_stop_bits="$(arg tool_stop_bits)"
+    tool_rx_idle_chars="$(arg tool_rx_idle_chars)"
+    tool_tx_idle_chars="$(arg tool_tx_idle_chars)"
+    tool_device_name="$(arg tool_device_name)"
+    tool_tcp_port="$(arg tool_tcp_port)"
+    robot_ip="$(arg robot_ip)"
+    script_filename="$(arg script_filename)"
+    output_recipe_filename="$(arg output_recipe_filename)"
+    input_recipe_filename="$(arg input_recipe_filename)"
+  >
+    <origin xyz="0 0 0" rpy="0 0 0" /> <!-- position robot in the world -->
+  </xacro:ur_robot>
+  <xacro:if value="$(arg sim_gazebo)">
     <!-- Gazebo plugins -->
-    <gazebo reference="world">
-    </gazebo>
+    <gazebo reference="world"></gazebo>
     <gazebo>
       <plugin filename="libgazebo_ros2_control.so" name="gazebo_ros2_control">
@@ -95,6 +96,5 @@
   <xacro:if value="$(arg sim_ignition)">
     <!-- Gazebo plugins -->
-    <gazebo reference="world">
-    </gazebo>
+    <gazebo reference="world"></gazebo>
     <gazebo>
       <plugin filename="libign_ros2_control-system.so" name="ign_ros2_control::IgnitionROS2ControlPlugin">
@@ -104,5 +104,9 @@
     </gazebo>
   </xacro:if>
+  <!-- table definition -->
+  <xacro:generate_table prefix="$(arg prefix)" attachment_link="world" table_name="robot_table"/>
+  <!-- manipulator definition -->
+  <xacro:generate_manipulator prefix="$(arg prefix)" attachment_link="tool0" manipulator_name="Klinke"/>
   <!-- camera definition -->
-  <xacro:generate_camera prefix="$(arg prefix)" attachment_link="tool0"/>
+  <!--xacro:generate_camera prefix="$(arg prefix)" attachment_link="tool0"/-->
 </robot>

File: ros2_ws/src/modproft_ur_moveit_config/srdf/ur.srdf.xacro (robot description, xacro)
@@ -5,5 +5,9 @@
   <!-- parameters -->
   <xacro:arg name="prefix" default="" />
-  <xacro:include filename="$(find ur_moveit_config)/srdf/ur_macro.srdf.xacro"/>
+  <xacro:include filename="$(find modproft_ur_moveit_config)/srdf/ur_macro.srdf.xacro"/>
   <xacro:ur_srdf name="$(arg name)" prefix="$(arg prefix)"/>
+  <disable_collisions link1="$(arg prefix)robot_table_link" link2="$(arg prefix)base_link" reason="Never" />
+  <disable_collisions link1="$(arg prefix)robot_table_tabletop_link" link2="$(arg prefix)base_link" reason="Adjacent" />
+  <disable_collisions link1="$(arg prefix)robot_table_tabletop_link" link2="$(arg prefix)base_link_inertia" reason="Adjacent" />
+  <disable_collisions link1="$(arg prefix)wrist_3_link" link2="$(arg prefix)Klinke_link" reason="Adjacent" />
 </robot>
